File: modules/macropad/PCB/cybdokeebs_macropad.kicad_sch (KiCad schematic)
At the start: 40 parts, among them SW10 SW_Push_45deg, SW11 SW_Push_45deg, SW12 SW_Push_45deg, SW13 SW_Push_45deg, SW14 SW_Push_45deg, SW15 SW_Push_45deg, SW16 SW_Push_45deg, SW17 SW_Push_45deg, SW18 SW_Push_45deg, SW19 SW_Push_45deg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

Commit message: macropad finished
Connections:
- net COL1 renamed GPIO18
- net GPIO18: now also SW15.1; no longer SW12.1
- net COL2 renamed GPIO17
- net GPIO17: now also SW12.1, SW16.1; no longer SW13.1, SW14.1
- net COL3 renamed GPIO14
- net GPIO14: now also SW13.1, SW17.1; no longer SW15.1, SW16.1
- net COL4 renamed GPIO11
- net GPIO11: now also SW14.1; no longer SW17.1
- net ROW1 renamed GPIO1
- net ROW2 renamed GPIO12
- net ROW3 renamed GPIO10
- net GPIO10: now also D10.1 (K), D12.1 (K); no longer D13.1 (K), D15.1 (K)
- net ROW4 renamed GPIO2
- net GPIO2: now also D13.1 (K), D15.1 (K); no longer D10.1 (K), D12.1 (K)
- net ROW5 renamed GPIO16
Other:
- moved on the sheet: D10, D11, D12, D13, D14, D15, SW12, SW13, SW14, SW15, SW16, SW17
