File: modules/macropad/PCB/minimum_system.kicad_sch (KiCad schematic)
At the start: 35 parts, among them J13 Conn_01x05_Socket, J14 Conn_01x05_Socket, J16 Conn_01x05_Pin, J9 Conn_01x05_Pin, SW1 BOOTSEL, SW2 RESET, U1 TCA4307DGKR, U2 RP2350_60QFN, U3 BM03B-SRSS-TB

Commit message: macropad finished
Parts:
- removed C16, C17: 100nF, Capacitor_SMD:C_0402_1005Metric_Pad0.74x0.62mm_HandSolder, symbol Device:C
- added J10, J15: Conn_01x05_Pin, imports:pogo 5pin 2.54, symbol Connector:Conn_01x05_Pin
- added J11, J12: Conn_01x05_Socket, imports:pogo 5pin 2.54, symbol Connector:Conn_01x05_Socket
- SW1: footprint Resistor_SMD:R_0402_1005Metric_Pad0.72x0.64mm_HandSolder -> Button_Switch_SMD:SW_Push_SPST_NO_Alps_SKRK
- SW2: value RESET -> BOOTSEL; footprint Resistor_SMD:R_0402_1005Metric_Pad0.72x0.64mm_HandSolder -> Button_Switch_SMD:SW_Push_SPST_NO_Alps_SKRK
- U1: footprint easyeda:VSSOP-8_L3.0-W3.0-P0.65-LS4.9-BL -> easyeda2kicad:VSSOP-8_L3.0-W3.0-P0.65-LS4.9-BL
Connections:
- net GPIO28 is gone; now on net SYS_SDA: U2.42 (GPIO28_ADC2)
- net GPIO29 is gone; now on net SYS_SCL: U2.43 (GPIO29_ADC3)
- net +3V3: now also J10.1 (Pin_1), J11.1 (Pin_1), J12.1 (Pin_1), J15.1 (Pin_1)
- net 0-0-SCL: now also J14.4 (Pin_4), J16.4 (Pin_4), J10.4 (Pin_4), J12.4 (Pin_4)
- net 0-0-SDA: now also J14.3 (Pin_3), J16.3 (Pin_3), J10.3 (Pin_3), J12.3 (Pin_3)
- net GND: now also J10.5 (Pin_5), J11.5 (Pin_5), J12.5 (Pin_5), J15.5 (Pin_5)
- net 0-0-EN: now reaches J14.2 (Pin_2), J16.2 (Pin_2)
- net 0-0-EN: now also J10.2 (Pin_2), J12.2 (Pin_2)
- net 0-1-EN: now reaches J13.2 (Pin_2), J9.2 (Pin_2)
- net 0-1-EN: now also J11.2 (Pin_2), J15.2 (Pin_2)
- net 0-1-SDA: now reaches J13.3 (Pin_3), J9.3 (Pin_3)
- net 0-1-SDA: now also J11.3 (Pin_3), J15.3 (Pin_3)
- net 0-1-SCL: now reaches J13.4 (Pin_4), J9.4 (Pin_4)
- net 0-1-SCL: now also J11.4 (Pin_4), J15.4 (Pin_4)
