File: modules/keyboard/PCB/minimum_system.kicad_sch (KiCad schematic)
At the start: 37 parts, among them J10 Conn_01x05_Pin, J11 Conn_01x05_Socket, J12 Conn_01x05_Socket, J13 Conn_01x05_Socket, J14 Conn_01x05_Socket, J15 Conn_01x05_Pin, J16 Conn_01x05_Pin, J9 Conn_01x05_Pin, SW1 BOOTSEL, SW2 BOOTSEL, U1 TCA4307DGKR, U2 RP2350_60QFN, U3 BM03B-SRSS-TB

Commit message: started main keyboard
Parts:
- removed J10, J15, J16, J9: Conn_01x05_Pin, imports:pogo 5pin 2.54, symbol Connector:Conn_01x05_Pin
- removed J13, J14: Conn_01x05_Socket, imports:pogo 5pin 2.54, symbol Connector:Conn_01x05_Socket
- added C11, C12: 100nF, Capacitor_SMD:C_0402_1005Metric_Pad0.74x0.62mm_HandSolder, symbol Device:C
- added J1, J2, J3, J4, J5, J7: Conn_01x05_Pin, imports:pogo 5pin 2.54, symbol Connector:Conn_01x05_Pin
- added J10, J6, J8, J9: Conn_01x05_Pin, imports:pogo 5pin 2.54, symbol Connector:Conn_01x05_Socket
- added R3, R5: 10kR, Resistor_SMD:R_0402_1005Metric_Pad0.72x0.64mm_HandSolder, symbol Device:R
- J11, J12: value Conn_01x05_Socket -> Conn_01x05_Pin
- L1: footprint imports:INDC1608X95N -> Resistor_SMD:R_0402_1005Metric_Pad0.72x0.64mm_HandSolder
- SW62: renamed from SW1; footprint Button_Switch_SMD:SW_Push_SPST_NO_Alps_SKRK -> PCM_Switch_Keyboard_Hotswap_Kailh:SW_Hotswap_Kailh_MX_plated_1.25u
- SW63: renamed from SW2; value BOOTSEL -> RESET; footprint Button_Switch_SMD:SW_Push_SPST_NO_Alps_SKRK -> PCM_Switch_Keyboard_Hotswap_Kailh:SW_Hotswap_Kailh_MX_plated_1.25u
- renumbered C8 to C1, C15 to C10, C3 to C13, C5 to C14, C4 to C15, C1 to C16, C2 to C17, C6 to C2, C7 to C3, C9 to C4, C10 to C5, C11 to C6, C12 to C7, C13 to C8, C14 to C9, R3 to R1, R9 to R8, R8 to R9
Connections:
- net +3V3: now also C11.2, C12.2, J1.1 (Pin_1), J10.1 (Pin_1), J2.1 (Pin_1), J3.1 (Pin_1), J4.1 (Pin_1), J4.2 (Pin_2), J5.1 (Pin_1), J6.1 (Pin_1), J6.2 (Pin_2), J7.1 (Pin_1), J7.2 (Pin_2), J8.1 (Pin_1), J9.1 (Pin_1), J9.2 (Pin_2), R3.1, R5.1
- net GND: now also C11.1, C12.1, J1.5 (Pin_5), J10.5 (Pin_5), J2.5 (Pin_5), J3.5 (Pin_5), J4.5 (Pin_5), J7.5 (Pin_5), J9.5 (Pin_5)
- net SYS_SCL: no longer U2.43 (GPIO29_ADC3)
- net SYS_SDA: no longer U2.42 (GPIO28_ADC2)
- net 0-0-EN renamed BUS2-EN
- net BUS2-EN: now also J3.2 (Pin_2); no longer U2.34 (GPIO22)
- net 0-0-SCL renamed BUS0-SCL
- net BUS0-SCL: now also J1.4 (Pin_4), J10.4 (Pin_4), J5.4 (Pin_4), R3.2; no longer J12.4 (Pin_4)
- net 0-0-SDA renamed BUS0-SDA
- net BUS0-SDA: now also J1.3 (Pin_3), J10.3 (Pin_3), J5.3 (Pin_3), R5.2; no longer J12.3 (Pin_3)
- net 0-1-EN renamed BUS1-EN
- net BUS1-EN: now also J2.2 (Pin_2)
- net 0-1-SCL renamed BUS1-SCL
- net BUS1-SCL: now also J2.4 (Pin_4)
- net 0-1-SDA renamed BUS1-SDA
- net BUS1-SDA: now also J2.3 (Pin_3)
- new net BUS0-EN: J1.2 (Pin_2), J10.2 (Pin_2), J5.2 (Pin_2)
- new net BUS2-SCL: J12.4 (Pin_4), J3.4 (Pin_4), J8.4 (Pin_4)
- new net BUS2-SDA: J12.3 (Pin_3), J3.3 (Pin_3), J8.2 (Pin_2), J8.3 (Pin_3)
- new net BUS3-SCL: J4.4 (Pin_4), J6.4 (Pin_4), J7.4 (Pin_4), J9.4 (Pin_4)
- new net BUS3-SDA: J4.3 (Pin_3), J6.3 (Pin_3), J7.3 (Pin_3), J9.3 (Pin_3)
- new net GPIO22: U2.34 (GPIO22)
- new net GPIO28: U2.42 (GPIO28_ADC2)
- new net GPIO29: U2.43 (GPIO29_ADC3)

Commit message: kb mostly done
Parts:
- removed C11, C12: 100nF, Capacitor_SMD:C_0402_1005Metric_Pad0.74x0.62mm_HandSolder, symbol Device:C
- removed R3, R5: 10kR, Resistor_SMD:R_0402_1005Metric_Pad0.72x0.64mm_HandSolder, symbol Device:R
- added J14, J15: Conn_01x05_Pin, imports:pogo 5pin 2.54, symbol Connector:Conn_01x05_Socket
- added J3, J4: Conn_01x05_Pin, imports:pogo 5pin 2.54, symbol Connector:Conn_01x05_Pin
- L1: footprint Resistor_SMD:R_0402_1005Metric_Pad0.72x0.64mm_HandSolder -> imports:INDC1608X95N
- SW1: renamed from SW62; footprint PCM_Switch_Keyboard_Hotswap_Kailh:SW_Hotswap_Kailh_MX_plated_1.25u -> Button_Switch_SMD:SW_Push_SPST_NO_Alps_SKRK
- SW2: renamed from SW63; footprint PCM_Switch_Keyboard_Hotswap_Kailh:SW_Hotswap_Kailh_MX_plated_1.25u -> Button_Switch_SMD:SW_Push_SPST_NO_Alps_SKRK
- renumbered J8 to J10, J9 to J11, J10 to J12, J11 to J13, J12 to J16, J3 to J5, J4 to J6, J5 to J7, J6 to J8, J7 to J9
Connections:
- net GPIO24 is gone; now on net SYS_SDA: U2.36 (GPIO24)
- net GPIO25 is gone; now on net SYS_SCL: U2.37 (GPIO25)
- net GPIO29 is gone; now on net BUS0-EN: U2.43 (GPIO29_ADC3)
- net +3V3: now also J14.1 (Pin_1), J15.1 (Pin_1), J3.1 (Pin_1), J4.1 (Pin_1); no longer J11.2 (Pin_2), J6.2 (Pin_2), J8.2 (Pin_2), J9.2 (Pin_2)
- net BUS2-EN: now also J14.2 (Pin_2), J3.2 (Pin_2); no longer J16.2 (Pin_2), J5.2 (Pin_2)
- net BUS2-SCL: now also J14.4 (Pin_4), J3.4 (Pin_4); no longer J10.4 (Pin_4), J16.4 (Pin_4), J5.4 (Pin_4)
- net BUS2-SDA: now also J14.3 (Pin_3), J3.3 (Pin_3); no longer J10.2 (Pin_2), J10.3 (Pin_3), J16.3 (Pin_3), J5.3 (Pin_3)
- net BUS3-SCL: now also J15.4 (Pin_4), J4.4 (Pin_4); no longer J11.4 (Pin_4), J6.4 (Pin_4), J8.4 (Pin_4), J9.4 (Pin_4)
- net BUS3-SDA: now also J15.3 (Pin_3), J4.3 (Pin_3); no longer J11.3 (Pin_3), J6.3 (Pin_3), J8.3 (Pin_3), J9.3 (Pin_3)
- net GND: now also J10.5 (Pin_5), J8.5 (Pin_5), J14.5 (Pin_5), J15.5 (Pin_5), J3.5 (Pin_5), J4.5 (Pin_5)
- new net BUS3-EN: J15.2 (Pin_2), J4.2 (Pin_2)
- new net BUS4-EN: J10.2 (Pin_2), J16.2 (Pin_2), J5.2 (Pin_2)
- new net BUS4-SCL: J10.4 (Pin_4), J16.4 (Pin_4), J5.4 (Pin_4)
- new net BUS4-SDA: J10.3 (Pin_3), J16.3 (Pin_3), J5.3 (Pin_3)
- new net BUS5-EN: J11.2 (Pin_2), J6.2 (Pin_2), J8.2 (Pin_2), J9.2 (Pin_2)
- new net BUS5-SCL: J11.4 (Pin_4), J6.4 (Pin_4), J8.4 (Pin_4), J9.4 (Pin_4)
- new net BUS5-SDA: J11.3 (Pin_3), J6.3 (Pin_3), J8.3 (Pin_3), J9.3 (Pin_3)
Other:
- moved on the sheet: J1, J10, J11, J12, J13, J16, J2, J5, J6, J7, J8, J9
