File: modules/keyboard/PCB/cybdokeebs_keyboard.kicad_pcb (KiCad board)
At the start: 2 copper layers, 173 parts, among them J1 Conn_01x05_Pin, J10 Conn_01x05_Pin, J11 Conn_01x05_Pin, J12 Conn_01x05_Pin, J2 Conn_01x05_Pin, J3 Conn_01x05_Pin, J4 Conn_01x05_Pin, J5 Conn_01x05_Pin, J6 Conn_01x05_Pin, J7 Conn_01x05_Pin, J8 Conn_01x05_Pin, J9 Conn_01x05_Pin, SW1 SW_Push, SW10 SW_Push, SW11 SW_Push, SW12 SW_Push, SW13 SW_Push, SW14 SW_Push, SW15 SW_Push, SW16 SW_Push, SW17 SW_Push, SW18 SW_Push, SW19 SW_Push, SW2 SW_Push, SW20 SW_Push, SW21 SW_Push, SW22 SW_Push, SW23 SW_Push, SW24 SW_Push, SW25 SW_Push, SW26 SW_Push, SW27 SW_Push, SW28 SW_Push, SW29 SW_Push, SW3 SW_Push, SW30 SW_Push, SW31 SW_Push, SW32 SW_Push, SW33 SW_Push, SW34 SW_Push, SW35 SW_Push, SW36 SW_Push, SW37 SW_Push, SW38 SW_Push, SW39 SW_Push, SW4 SW_Push, SW40 SW_Push, SW41 SW_Push, SW42 SW_Push, SW43 SW_Push, SW44 SW_Push, SW45 SW_Push, SW46 SW_Push, SW47 SW_Push, SW48 SW_Push, SW49 SW_Push, SW5 SW_Push, SW50 SW_Push, SW51 SW_Push, SW52 SW_Push, SW53 SW_Push, SW54 SW_Push, SW55 SW_Push, SW56 SW_Push, SW57 SW_Push, SW58 SW_Push, SW59 SW_Push, SW6 SW_Push, SW60 SW_Push, SW61 SW_Push, SW62 BOOTSEL, SW63 RESET, SW7 SW_Push, SW8 SW_Push, SW9 SW_Push, U1 TCA4307DGKR, U2 RP2350_60QFN, U3 BM03B-SRSS-TB

Commit message: kb mostly done
Parts:
- removed C11, C12: 100nF, Capacitor_SMD:C_0402_1005Metric_Pad0.74x0.62mm_HandSolder
- removed R3, R5: 10kR, Resistor_SMD:R_0402_1005Metric_Pad0.72x0.64mm_HandSolder
- removed the U1 at (-41.9, -6.97)
- added J14: Conn_01x05_Pin, imports:pogo 5pin 2.54, F.Cu at (219.2, 230.9)
- added J15: Conn_01x05_Pin, imports:pogo 5pin 2.54, F.Cu at (269.2, 230.9)
- added J3: Conn_01x05_Pin, imports:pogo 5pin 2.54, F.Cu at (169.2, 121.9)
- added J4: Conn_01x05_Pin, imports:pogo 5pin 2.54, F.Cu at (219.2, 121.9)
- C1, C10, C13, C14, C15, C16, C17, C2, C3, C4, C5, C6, C7, C8, C9, D1, D10, D11, D12, D13, D14, D15, D16, D17, D18, D19, D2, D20, D21, D22, D23, D24, D25, D26, D27, D28, D29, D3, D30, D31, D32, D33, D34, D35, D36, D37, D38, D39, D4, D40, D41, D5, D53, D6, D7, D8, D9, R1, R10, R2, R4, R6, R7, R8, R9, U1, U2, U3: moved to B.Cu
- D42: renamed from D52; moved to B.Cu
- D43: renamed from D42; moved to B.Cu
- D44: renamed from D43; moved to B.Cu
- D45: renamed from D44; moved to B.Cu
- D46: renamed from D45; moved to B.Cu
- D47: renamed from D46; moved to B.Cu
- D48: renamed from D47; moved to B.Cu
- D49: renamed from D48; moved to B.Cu
- D50: renamed from D49; moved to B.Cu
- D51: renamed from D50; moved to B.Cu
- D52: renamed from D51; moved to B.Cu
- D54: renamed from D55; moved to B.Cu
- D55: renamed from D56; moved to B.Cu
- D56: renamed from D57; moved to B.Cu
- D57: renamed from D58; moved to B.Cu
- D58: renamed from D59; moved to B.Cu
- D59: renamed from D60; moved to B.Cu
- D60: renamed from D61; moved to B.Cu
- D61: renamed from D54; moved to B.Cu
- L1: footprint Resistor_SMD:R_0402_1005Metric_Pad0.72x0.64mm_HandSolder -> imports:INDC1608X95N; moved to B.Cu
- SW1: renamed from SW62; footprint PCM_Switch_Keyboard_Hotswap_Kailh:SW_Hotswap_Kailh_MX_plated_1.25u -> Button_Switch_SMD:SW_Push_SPST_NO_Alps_SKRK; moved to B.Cu
- SW10: renamed from SW8; footprint PCM_Switch_Keyboard_Hotswap_Kailh:SW_Hotswap_Kailh_MX_plated_1.00u -> PCM_Switch_Keyboard_Hotswap_Kailh:SW_Hotswap_Kailh_MX_1.00u
- SW11: renamed from SW9; footprint PCM_Switch_Keyboard_Hotswap_Kailh:SW_Hotswap_Kailh_MX_plated_1.00u -> PCM_Switch_Keyboard_Hotswap_Kailh:SW_Hotswap_Kailh_MX_1.00u
- SW12: renamed from SW10; footprint PCM_Switch_Keyboard_Hotswap_Kailh:SW_Hotswap_Kailh_MX_plated_1.00u -> PCM_Switch_Keyboard_Hotswap_Kailh:SW_Hotswap_Kailh_MX_1.00u
- SW13: renamed from SW11; footprint PCM_Switch_Keyboard_Hotswap_Kailh:SW_Hotswap_Kailh_MX_plated_1.00u -> PCM_Switch_Keyboard_Hotswap_Kailh:SW_Hotswap_Kailh_MX_1.00u
- SW14: renamed from SW12; footprint PCM_Switch_Keyboard_Hotswap_Kailh:SW_Hotswap_Kailh_MX_plated_1.00u -> PCM_Switch_Keyboard_Hotswap_Kailh:SW_Hotswap_Kailh_MX_1.00u
- SW15: renamed from SW13; footprint PCM_Switch_Keyboard_Hotswap_Kailh:SW_Hotswap_Kailh_MX_plated_1.00u -> PCM_Switch_Keyboard_Hotswap_Kailh:SW_Hotswap_Kailh_MX_1.00u
- SW16: renamed from SW14; footprint PCM_Switch_Keyboard_Hotswap_Kailh:SW_Hotswap_Kailh_MX_plated_1.00u -> PCM_Switch_Keyboard_Hotswap_Kailh:SW_Hotswap_Kailh_MX_2.00u
- SW17: renamed from SW15; footprint PCM_Switch_Keyboard_Hotswap_Kailh:SW_Hotswap_Kailh_MX_plated_1.00u -> PCM_Switch_Keyboard_Hotswap_Kailh:SW_Hotswap_Kailh_MX_1.50u
- SW18: renamed from SW16; footprint PCM_Switch_Keyboard_Hotswap_Kailh:SW_Hotswap_Kailh_MX_plated_2.00u -> PCM_Switch_Keyboard_Hotswap_Kailh:SW_Hotswap_Kailh_MX_1.00u
- SW19: renamed from SW17; footprint PCM_Switch_Keyboard_Hotswap_Kailh:SW_Hotswap_Kailh_MX_plated_1.50u -> PCM_Switch_Keyboard_Hotswap_Kailh:SW_Hotswap_Kailh_MX_1.00u
- SW2: renamed from SW63; footprint PCM_Switch_Keyboard_Hotswap_Kailh:SW_Hotswap_Kailh_MX_plated_1.25u -> Button_Switch_SMD:SW_Push_SPST_NO_Alps_SKRK; moved to B.Cu
- SW20: renamed from SW18; footprint PCM_Switch_Keyboard_Hotswap_Kailh:SW_Hotswap_Kailh_MX_plated_1.00u -> PCM_Switch_Keyboard_Hotswap_Kailh:SW_Hotswap_Kailh_MX_1.00u
- SW21: renamed from SW19; footprint PCM_Switch_Keyboard_Hotswap_Kailh:SW_Hotswap_Kailh_MX_plated_1.00u -> PCM_Switch_Keyboard_Hotswap_Kailh:SW_Hotswap_Kailh_MX_1.00u
- SW22: renamed from SW20; footprint PCM_Switch_Keyboard_Hotswap_Kailh:SW_Hotswap_Kailh_MX_plated_1.00u -> PCM_Switch_Keyboard_Hotswap_Kailh:SW_Hotswap_Kailh_MX_1.00u
- SW23: renamed from SW21; footprint PCM_Switch_Keyboard_Hotswap_Kailh:SW_Hotswap_Kailh_MX_plated_1.00u -> PCM_Switch_Keyboard_Hotswap_Kailh:SW_Hotswap_Kailh_MX_1.00u
- SW24: renamed from SW22; footprint PCM_Switch_Keyboard_Hotswap_Kailh:SW_Hotswap_Kailh_MX_plated_1.00u -> PCM_Switch_Keyboard_Hotswap_Kailh:SW_Hotswap_Kailh_MX_1.00u
- SW25: renamed from SW23; footprint PCM_Switch_Keyboard_Hotswap_Kailh:SW_Hotswap_Kailh_MX_plated_1.00u -> PCM_Switch_Keyboard_Hotswap_Kailh:SW_Hotswap_Kailh_MX_1.00u
- SW26: renamed from SW24; footprint PCM_Switch_Keyboard_Hotswap_Kailh:SW_Hotswap_Kailh_MX_plated_1.00u -> PCM_Switch_Keyboard_Hotswap_Kailh:SW_Hotswap_Kailh_MX_1.00u
- SW27: renamed from SW25; footprint PCM_Switch_Keyboard_Hotswap_Kailh:SW_Hotswap_Kailh_MX_plated_1.00u -> PCM_Switch_Keyboard_Hotswap_Kailh:SW_Hotswap_Kailh_MX_1.00u
- SW28: renamed from SW26; footprint PCM_Switch_Keyboard_Hotswap_Kailh:SW_Hotswap_Kailh_MX_plated_1.00u -> PCM_Switch_Keyboard_Hotswap_Kailh:SW_Hotswap_Kailh_MX_1.00u
- SW29: renamed from SW27; footprint PCM_Switch_Keyboard_Hotswap_Kailh:SW_Hotswap_Kailh_MX_plated_1.00u -> PCM_Switch_Keyboard_Hotswap_Kailh:SW_Hotswap_Kailh_MX_1.00u
- SW3: renamed from SW1; footprint Button_Switch_SMD:SW_Push_SPST_NO_Alps_SKRK -> PCM_Switch_Keyboard_Hotswap_Kailh:SW_Hotswap_Kailh_MX_1.00u
- SW30: renamed from SW28; footprint PCM_Switch_Keyboard_Hotswap_Kailh:SW_Hotswap_Kailh_MX_plated_1.00u -> PCM_Switch_Keyboard_Hotswap_Kailh:SW_Hotswap_Kailh_MX_1.50u
- SW31: renamed from SW29; footprint PCM_Switch_Keyboard_Hotswap_Kailh:SW_Hotswap_Kailh_MX_plated_1.00u -> PCM_Switch_Keyboard_Hotswap_Kailh:SW_Hotswap_Kailh_MX_1.75u
- SW32: renamed from SW30; footprint PCM_Switch_Keyboard_Hotswap_Kailh:SW_Hotswap_Kailh_MX_plated_1.00u -> PCM_Switch_Keyboard_Hotswap_Kailh:SW_Hotswap_Kailh_MX_1.00u
- SW33: renamed from SW31; footprint PCM_Switch_Keyboard_Hotswap_Kailh:SW_Hotswap_Kailh_MX_plated_1.75u -> PCM_Switch_Keyboard_Hotswap_Kailh:SW_Hotswap_Kailh_MX_1.00u
- SW34: renamed from SW32; footprint PCM_Switch_Keyboard_Hotswap_Kailh:SW_Hotswap_Kailh_MX_plated_1.00u -> PCM_Switch_Keyboard_Hotswap_Kailh:SW_Hotswap_Kailh_MX_1.00u
- SW35: renamed from SW33; footprint PCM_Switch_Keyboard_Hotswap_Kailh:SW_Hotswap_Kailh_MX_plated_1.00u -> PCM_Switch_Keyboard_Hotswap_Kailh:SW_Hotswap_Kailh_MX_1.00u
- SW36: renamed from SW34; footprint PCM_Switch_Keyboard_Hotswap_Kailh:SW_Hotswap_Kailh_MX_plated_1.00u -> PCM_Switch_Keyboard_Hotswap_Kailh:SW_Hotswap_Kailh_MX_1.00u
- SW37: renamed from SW35; footprint PCM_Switch_Keyboard_Hotswap_Kailh:SW_Hotswap_Kailh_MX_plated_1.00u -> PCM_Switch_Keyboard_Hotswap_Kailh:SW_Hotswap_Kailh_MX_1.00u
- SW38: renamed from SW36; footprint PCM_Switch_Keyboard_Hotswap_Kailh:SW_Hotswap_Kailh_MX_plated_1.00u -> PCM_Switch_Keyboard_Hotswap_Kailh:SW_Hotswap_Kailh_MX_1.00u
- SW39: renamed from SW37; footprint PCM_Switch_Keyboard_Hotswap_Kailh:SW_Hotswap_Kailh_MX_plated_1.00u -> PCM_Switch_Keyboard_Hotswap_Kailh:SW_Hotswap_Kailh_MX_1.00u
- SW4: renamed from SW2; footprint Button_Switch_SMD:SW_Push_SPST_NO_Alps_SKRK -> PCM_Switch_Keyboard_Hotswap_Kailh:SW_Hotswap_Kailh_MX_1.00u
- SW40: renamed from SW38; footprint PCM_Switch_Keyboard_Hotswap_Kailh:SW_Hotswap_Kailh_MX_plated_1.00u -> PCM_Switch_Keyboard_Hotswap_Kailh:SW_Hotswap_Kailh_MX_1.00u
- SW41: renamed from SW39; footprint PCM_Switch_Keyboard_Hotswap_Kailh:SW_Hotswap_Kailh_MX_plated_1.00u -> PCM_Switch_Keyboard_Hotswap_Kailh:SW_Hotswap_Kailh_MX_1.00u
- SW42: renamed from SW40; footprint PCM_Switch_Keyboard_Hotswap_Kailh:SW_Hotswap_Kailh_MX_plated_1.00u -> PCM_Switch_Keyboard_Hotswap_Kailh:SW_Hotswap_Kailh_MX_1.00u
- SW43: renamed from SW41; footprint PCM_Switch_Keyboard_Hotswap_Kailh:SW_Hotswap_Kailh_MX_plated_1.00u -> PCM_Switch_Keyboard_Hotswap_Kailh:SW_Hotswap_Kailh_MX_2.25u
- SW44: renamed from SW52; footprint PCM_Switch_Keyboard_Hotswap_Kailh:SW_Hotswap_Kailh_MX_plated_1.00u -> PCM_Switch_Keyboard_Hotswap_Kailh:SW_Hotswap_Kailh_MX_2.25u
- SW45: renamed from SW42; footprint PCM_Switch_Keyboard_Hotswap_Kailh:SW_Hotswap_Kailh_MX_plated_1.00u -> PCM_Switch_Keyboard_Hotswap_Kailh:SW_Hotswap_Kailh_MX_1.00u
- SW46: renamed from SW43; footprint PCM_Switch_Keyboard_Hotswap_Kailh:SW_Hotswap_Kailh_MX_plated_2.25u -> PCM_Switch_Keyboard_Hotswap_Kailh:SW_Hotswap_Kailh_MX_1.00u
- SW47: renamed from SW44; footprint PCM_Switch_Keyboard_Hotswap_Kailh:SW_Hotswap_Kailh_MX_plated_2.25u -> PCM_Switch_Keyboard_Hotswap_Kailh:SW_Hotswap_Kailh_MX_1.00u
- SW48: renamed from SW45; footprint PCM_Switch_Keyboard_Hotswap_Kailh:SW_Hotswap_Kailh_MX_plated_1.00u -> PCM_Switch_Keyboard_Hotswap_Kailh:SW_Hotswap_Kailh_MX_1.00u
- SW49: renamed from SW46; footprint PCM_Switch_Keyboard_Hotswap_Kailh:SW_Hotswap_Kailh_MX_plated_1.00u -> PCM_Switch_Keyboard_Hotswap_Kailh:SW_Hotswap_Kailh_MX_1.00u
- SW5: renamed from SW3; footprint PCM_Switch_Keyboard_Hotswap_Kailh:SW_Hotswap_Kailh_MX_plated_1.00u -> PCM_Switch_Keyboard_Hotswap_Kailh:SW_Hotswap_Kailh_MX_1.00u
- SW50: renamed from SW47; footprint PCM_Switch_Keyboard_Hotswap_Kailh:SW_Hotswap_Kailh_MX_plated_1.00u -> PCM_Switch_Keyboard_Hotswap_Kailh:SW_Hotswap_Kailh_MX_1.00u
- SW51: renamed from SW48; footprint PCM_Switch_Keyboard_Hotswap_Kailh:SW_Hotswap_Kailh_MX_plated_1.00u -> PCM_Switch_Keyboard_Hotswap_Kailh:SW_Hotswap_Kailh_MX_1.00u
- SW52: renamed from SW49; footprint PCM_Switch_Keyboard_Hotswap_Kailh:SW_Hotswap_Kailh_MX_plated_1.00u -> PCM_Switch_Keyboard_Hotswap_Kailh:SW_Hotswap_Kailh_MX_1.00u
- SW53: renamed from SW50; footprint PCM_Switch_Keyboard_Hotswap_Kailh:SW_Hotswap_Kailh_MX_plated_1.00u -> PCM_Switch_Keyboard_Hotswap_Kailh:SW_Hotswap_Kailh_MX_1.00u
- SW54: renamed from SW51; footprint PCM_Switch_Keyboard_Hotswap_Kailh:SW_Hotswap_Kailh_MX_plated_1.00u -> PCM_Switch_Keyboard_Hotswap_Kailh:SW_Hotswap_Kailh_MX_1.00u
- SW55: renamed from SW53; footprint PCM_Switch_Keyboard_Hotswap_Kailh:SW_Hotswap_Kailh_MX_plated_1.00u -> PCM_Switch_Keyboard_Hotswap_Kailh:SW_Hotswap_Kailh_MX_2.75u
- SW56: renamed from SW55; footprint PCM_Switch_Keyboard_Hotswap_Kailh:SW_Hotswap_Kailh_MX_plated_2.75u -> PCM_Switch_Keyboard_Hotswap_Kailh:SW_Hotswap_Kailh_MX_1.25u
- SW57: renamed from SW56; footprint PCM_Switch_Keyboard_Hotswap_Kailh:SW_Hotswap_Kailh_MX_plated_1.25u -> PCM_Switch_Keyboard_Hotswap_Kailh:SW_Hotswap_Kailh_MX_1.25u
- SW58: renamed from SW57; footprint PCM_Switch_Keyboard_Hotswap_Kailh:SW_Hotswap_Kailh_MX_plated_1.25u -> PCM_Switch_Keyboard_Hotswap_Kailh:SW_Hotswap_Kailh_MX_1.25u
- SW59: renamed from SW58; footprint PCM_Switch_Keyboard_Hotswap_Kailh:SW_Hotswap_Kailh_MX_plated_1.25u -> PCM_Switch_Keyboard_Hotswap_Kailh:SW_Hotswap_Kailh_MX_6.25u
- SW6: renamed from SW4; footprint PCM_Switch_Keyboard_Hotswap_Kailh:SW_Hotswap_Kailh_MX_plated_1.00u -> PCM_Switch_Keyboard_Hotswap_Kailh:SW_Hotswap_Kailh_MX_1.00u
- SW60: renamed from SW59; footprint PCM_Switch_Keyboard_Hotswap_Kailh:SW_Hotswap_Kailh_MX_plated_6.25u -> PCM_Switch_Keyboard_Hotswap_Kailh:SW_Hotswap_Kailh_MX_1.25u
- SW61: renamed from SW60; footprint PCM_Switch_Keyboard_Hotswap_Kailh:SW_Hotswap_Kailh_MX_plated_1.25u -> PCM_Switch_Keyboard_Hotswap_Kailh:SW_Hotswap_Kailh_MX_1.25u
- SW62: renamed from SW61; footprint PCM_Switch_Keyboard_Hotswap_Kailh:SW_Hotswap_Kailh_MX_plated_1.25u -> PCM_Switch_Keyboard_Hotswap_Kailh:SW_Hotswap_Kailh_MX_1.25u
- SW63: renamed from SW54; footprint PCM_Switch_Keyboard_Hotswap_Kailh:SW_Hotswap_Kailh_MX_plated_1.00u -> PCM_Switch_Keyboard_Hotswap_Kailh:SW_Hotswap_Kailh_MX_1.25u
- SW7: renamed from SW5; footprint PCM_Switch_Keyboard_Hotswap_Kailh:SW_Hotswap_Kailh_MX_plated_1.00u -> PCM_Switch_Keyboard_Hotswap_Kailh:SW_Hotswap_Kailh_MX_1.00u
- SW8: renamed from SW6; footprint PCM_Switch_Keyboard_Hotswap_Kailh:SW_Hotswap_Kailh_MX_plated_1.00u -> PCM_Switch_Keyboard_Hotswap_Kailh:SW_Hotswap_Kailh_MX_1.00u
- SW9: renamed from SW7; footprint PCM_Switch_Keyboard_Hotswap_Kailh:SW_Hotswap_Kailh_MX_plated_1.00u -> PCM_Switch_Keyboard_Hotswap_Kailh:SW_Hotswap_Kailh_MX_1.00u
- moved J8 502.5 mm to (341.2, 143.9), turned to -90 degrees
- moved J10 502.0 mm to (341.2, 203.9), turned to -90 degrees
- moved J6 481.9 mm to (319.2, 121.9)
- moved J16 480.9 mm to (319.2, 230.9)
- moved SW16 464.5 mm to (320.5, 138.0)
- moved SW30 445.6 mm to (325.2, 157.0)
- moved SW15 439.7 mm to (291.9, 138.0)
- moved J5 431.9 mm to (269.2, 121.9)
- moved SW14 430.0 mm to (272.8, 138.0)
- moved SW29 423.1 mm to (301.4, 157.0)
- moved SW43 422.7 mm to (318.1, 176.1)
- moved SW63 409.4 mm to (327.6, 214.2)
- moved SW13 406.8 mm to (253.8, 138.0)
- moved SW28 406.0 mm to (282.4, 157.0)
- moved SW42 398.3 mm to (287.1, 176.1)
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- renumbered H4 to H3, H3 to H4, J8 to J10, J9 to J11, J10 to J12, J11 to J13, J12 to J16, J3 to J5, J4 to J6, J5 to J7, J6 to J8, J7 to J9
Connections:
- net /minimum_system/BUS2-SCL renamed /minimum_system/BUS4-SCL
- net /minimum_system/BUS3-SCL renamed /minimum_system/BUS5-SCL
- net /minimum_system/BUS3-SDA renamed /minimum_system/BUS5-SDA
- D1 pad 1: Net-(D1-K) -> GPIO13
- D10 pad 1: Net-(D1-K) -> GPIO13
- D11 pad 1: Net-(D1-K) -> GPIO13
- D12 pad 1: Net-(D1-K) -> GPIO13
- D13 pad 1: Net-(D1-K) -> GPIO13
- D14 pad 1: Net-(D1-K) -> GPIO13
- D15 pad 1: Net-(D15-K) -> GPIO12
- D16 pad 1: Net-(D15-K) -> GPIO12
- D17 pad 1: Net-(D15-K) -> GPIO12
- D18 pad 1: Net-(D15-K) -> GPIO12
- D19 pad 1: Net-(D15-K) -> GPIO12
- D2 pad 1: Net-(D1-K) -> GPIO13
- D20 pad 1: Net-(D15-K) -> GPIO12
- D21 pad 1: Net-(D15-K) -> GPIO12
- D22 pad 1: Net-(D15-K) -> GPIO12
- D23 pad 1: Net-(D15-K) -> GPIO12
- D24 pad 1: Net-(D15-K) -> GPIO12
- D25 pad 1: Net-(D15-K) -> GPIO12
- D26 pad 1: Net-(D15-K) -> GPIO12
- D27 pad 1: Net-(D15-K) -> GPIO12
- D28 pad 1: Net-(D15-K) -> GPIO12
- D29 pad 1: Net-(D29-K) -> GPIO11
- D3 pad 1: Net-(D1-K) -> GPIO13
- D30 pad 1: Net-(D29-K) -> GPIO11
- D31 pad 1: Net-(D29-K) -> GPIO11
- D32 pad 1: Net-(D29-K) -> GPIO11
- D33 pad 1: Net-(D29-K) -> GPIO11
- D34 pad 1: Net-(D29-K) -> GPIO11
- D35 pad 1: Net-(D29-K) -> GPIO11
- D36 pad 1: Net-(D29-K) -> GPIO11
- D37 pad 1: Net-(D29-K) -> GPIO11
- D38 pad 1: Net-(D29-K) -> GPIO11
- D39 pad 1: Net-(D29-K) -> GPIO11
- D4 pad 1: Net-(D1-K) -> GPIO13
- D40 pad 1: Net-(D29-K) -> GPIO11
- D41 pad 1: Net-(D29-K) -> GPIO11
- D42 pad 1: Net-(D42-K) -> GPIO9
- D43 pad 1: Net-(D42-K) -> GPIO9
- D44 pad 1: Net-(D42-K) -> GPIO9
- D45 pad 1: Net-(D42-K) -> GPIO9
- D46 pad 1: Net-(D42-K) -> GPIO9
- D47 pad 1: Net-(D42-K) -> GPIO9
- D48 pad 1: Net-(D42-K) -> GPIO9
- D49 pad 1: Net-(D42-K) -> GPIO9
- D5 pad 1: Net-(D1-K) -> GPIO13
- D50 pad 1: Net-(D42-K) -> GPIO9
- D51 pad 1: Net-(D42-K) -> GPIO9
- D52 pad 1: Net-(D42-K) -> GPIO9
- D53 pad 1: Net-(D42-K) -> GPIO9
- D54 pad 1: Net-(D54-K) -> GPIO8
- D55 pad 1: Net-(D54-K) -> GPIO8
- D56 pad 1: Net-(D54-K) -> GPIO8
- D57 pad 1: Net-(D54-K) -> GPIO8
- D58 pad 1: Net-(D54-K) -> GPIO8
- D59 pad 1: Net-(D54-K) -> GPIO8
- D6 pad 1: Net-(D1-K) -> GPIO13
- D60 pad 1: Net-(D54-K) -> GPIO8
- D61 pad 1: Net-(D54-K) -> GPIO8
- D7 pad 1: Net-(D1-K) -> GPIO13
- D8 pad 1: Net-(D1-K) -> GPIO13
- D9 pad 1: Net-(D1-K) -> GPIO13
- J10 pad 2: /minimum_system/BUS2-SDA -> /minimum_system/BUS4-EN
- J10 pad 3: /minimum_system/BUS2-SDA -> /minimum_system/BUS4-SDA
- J10 pad 5: unconnected-(J8-Pin_5-Pad5) -> GND
- J11 pad 2: +3V3 -> /minimum_system/BUS5-EN
- J16 pad 2: /minimum_system/BUS2-EN -> /minimum_system/BUS4-EN
- J16 pad 3: /minimum_system/BUS2-SDA -> /minimum_system/BUS4-SDA
- J5 pad 2: /minimum_system/BUS2-EN -> /minimum_system/BUS4-EN
- J5 pad 3: /minimum_system/BUS2-SDA -> /minimum_system/BUS4-SDA
- J6 pad 2: +3V3 -> /minimum_system/BUS5-EN
- J8 pad 2: +3V3 -> /minimum_system/BUS5-EN
- J8 pad 5: unconnected-(J6-Pin_5-Pad5) -> GND
- J9 pad 2: +3V3 -> /minimum_system/BUS5-EN
- SW10 pad 1: Net-(SW22-Pad1) -> GPIO16
- SW11 pad 1: Net-(SW23-Pad1) -> GPIO17
- SW12 pad 1: Net-(SW10-Pad1) -> GPIO19
- SW13 pad 1: Net-(SW11-Pad1) -> GPIO20
- SW14 pad 1: Net-(SW12-Pad1) -> GPIO21
- SW15 pad 1: Net-(SW13-Pad1) -> GPIO18
- SW16 pad 1: Net-(SW14-Pad1) -> GPIO22
- SW17 pad 1: Net-(SW1-Pad1) -> GPIO0
- SW18 pad 1: Net-(SW16-Pad1) -> GPIO1
- SW19 pad 1: Net-(SW17-Pad1) -> GPIO2
- SW20 pad 1: Net-(SW18-Pad1) -> GPIO3
- SW21 pad 1: Net-(SW19-Pad1) -> GPIO10
- SW22 pad 1: Net-(SW20-Pad1) -> GPIO14
- SW23 pad 1: Net-(SW21-Pad1) -> GPIO15
- SW24 pad 1: Net-(SW22-Pad1) -> GPIO16
- SW25 pad 1: Net-(SW23-Pad1) -> GPIO17
- SW26 pad 1: Net-(SW10-Pad1) -> GPIO19
- SW27 pad 1: Net-(SW11-Pad1) -> GPIO20
- SW28 pad 1: Net-(SW12-Pad1) -> GPIO21
- SW29 pad 1: Net-(SW13-Pad1) -> GPIO18
- SW3 pad 1: Net-(SW1-Pad1) -> GPIO0
- SW30 pad 1: Net-(SW14-Pad1) -> GPIO22
- SW31 pad 1: Net-(SW1-Pad1) -> GPIO0
- SW32 pad 1: Net-(SW16-Pad1) -> GPIO1
- SW33 pad 1: Net-(SW17-Pad1) -> GPIO2
- SW34 pad 1: Net-(SW18-Pad1) -> GPIO3
- SW35 pad 1: Net-(SW19-Pad1) -> GPIO10
- SW36 pad 1: Net-(SW20-Pad1) -> GPIO14
- SW37 pad 1: Net-(SW21-Pad1) -> GPIO15
- SW38 pad 1: Net-(SW22-Pad1) -> GPIO16
- SW39 pad 1: Net-(SW23-Pad1) -> GPIO17
- SW4 pad 1: Net-(SW16-Pad1) -> GPIO1
- SW40 pad 1: Net-(SW10-Pad1) -> GPIO19
- SW41 pad 1: Net-(SW11-Pad1) -> GPIO20
- SW42 pad 1: Net-(SW12-Pad1) -> GPIO21
- SW43 pad 1: Net-(SW14-Pad1) -> GPIO22
- SW44 pad 1: Net-(SW1-Pad1) -> GPIO0
- SW45 pad 1: Net-(SW16-Pad1) -> GPIO1
- SW46 pad 1: Net-(SW17-Pad1) -> GPIO2
- SW47 pad 1: Net-(SW18-Pad1) -> GPIO3
- SW48 pad 1: Net-(SW19-Pad1) -> GPIO10
- SW49 pad 1: Net-(SW20-Pad1) -> GPIO14
- SW5 pad 1: Net-(SW17-Pad1) -> GPIO2
- SW50 pad 1: Net-(SW21-Pad1) -> GPIO15
- SW51 pad 1: Net-(SW22-Pad1) -> GPIO16
- SW52 pad 1: Net-(SW23-Pad1) -> GPIO17
- SW53 pad 1: Net-(SW10-Pad1) -> GPIO19
- SW54 pad 1: Net-(SW11-Pad1) -> GPIO20
- SW55 pad 1: Net-(SW14-Pad1) -> GPIO22
- SW56 pad 1: Net-(SW1-Pad1) -> GPIO0
- SW57 pad 1: Net-(SW16-Pad1) -> GPIO1
- SW58 pad 1: Net-(SW17-Pad1) -> GPIO2
- SW59 pad 1: Net-(D42-K) -> GPIO14
- SW6 pad 1: Net-(SW18-Pad1) -> GPIO3
- SW60 pad 1: Net-(SW10-Pad1) -> GPIO19
- SW61 pad 1: Net-(SW11-Pad1) -> GPIO20
- SW62 pad 1: Net-(SW12-Pad1) -> GPIO21
- SW63 pad 1: Net-(SW14-Pad1) -> GPIO22
- SW7 pad 1: Net-(SW19-Pad1) -> GPIO10
- SW8 pad 1: Net-(SW20-Pad1) -> GPIO14
- SW9 pad 1: Net-(SW21-Pad1) -> GPIO15
- U2 pad 36: GPIO24 -> /minimum_system/SYS_SDA
- U2 pad 37: GPIO25 -> /minimum_system/SYS_SCL
- U2 pad 43: GPIO29 -> /minimum_system/BUS0-EN
Routing:
- net +3V3: track 0.00 -> 932.0 mm, vias 0 -> 5
- net GPIO13: track 0.00 -> 357.3 mm
- net GPIO12: track 0.00 -> 350.7 mm, vias 0 -> 26
- net /minimum_system/BUS5-SCL: track 0.00 -> 336.9 mm
- net /minimum_system/BUS5-SDA: track 0.00 -> 323.9 mm, vias 0 -> 4
- net /minimum_system/BUS5-EN: track 0.00 -> 322.7 mm, vias 0 -> 3
- net GPIO11: track 0.00 -> 320.2 mm, vias 0 -> 26
- net GPIO22: track 0.00 -> 271.0 mm
- net GPIO21: track 0.00 -> 243.4 mm
- net GPIO8: track 0.00 -> 240.5 mm, vias 0 -> 14
- net GPIO18: track 0.00 -> 237.2 mm, vias 0 -> 4
- net GPIO20: track 0.00 -> 218.9 mm
- net /minimum_system/BUS0-EN: track 0.00 -> 210.9 mm, vias 0 -> 2
- net /minimum_system/BUS0-SCL: track 0.00 -> 209.3 mm
- net /minimum_system/BUS0-SDA: track 0.00 -> 207.8 mm
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- added copper zone on B.Cu, net GND
- added copper zone on F.Cu, net GND
Other:
- board outline added: 294 x 114 mm

Commit message: finished all pcbs
Parts:
- added ?: , , F.Cu at (302.4, 138.3)
- added ?: , , F.Cu at (302.6, 228.2)
- added ?: , , F.Cu at (84.0, 174.8)
- added REF**: MountingHole_3.2mm_M3, MountingHole:MountingHole_3.2mm_M3, F.Cu at (98.8, 228.0)
- moved C4 1.01 mm to (145.1, 211.6)
Routing:
- net GPIO9: track 29.3 -> 282.0 mm, vias 0 -> 28
- net /minimum_system/BUS5-SDA: track 323.9 -> 418.7 mm, vias 4 -> 5
- net /minimum_system/BUS5-EN: track 322.7 -> 417.3 mm, vias 3 -> 4
- net /minimum_system/BUS5-SCL: track 336.9 -> 425.3 mm, vias 0 -> 1
- net /minimum_system/BOOTSEL: track 4.23 -> 66.9 mm, vias 1 -> 4
- net GPIO8: track 240.5 -> 290.4 mm, vias 14 -> 18
- net +3V3: track 932.0 -> 974.6 mm, vias 5 -> 7
- net /minimum_system/RESET: track 50.9 -> 53.1 mm
- net /minimum_system/SWDIO: track 59.4 -> 61.6 mm
- net /minimum_system/SWCLK: track 59.4 -> 61.7 mm
- net GND: vias 192 -> 252
