File: modules/controller_hub/pcb/CybdoKeebs_hub.kicad_pcb (KiCad board)
At the start: 2 copper layers, 14 parts, among them U1 RP2350_60QFN, U3 USBLC6-2P6, U4 USBLC6-2P6, U5 USBLC6-2P6, U6 USBLC6-2P6, U7 MCP1700x-300xxTT

Commit message: hub done, started macropad
Parts:
- added C1: 15pF, Capacitor_SMD:C_0402_1005Metric_Pad0.74x0.62mm_HandSolder, F.Cu at (179.6, 144.0)
- added C10: 100nF, Capacitor_SMD:C_0402_1005Metric_Pad0.74x0.62mm_HandSolder, F.Cu at (175.1, 139.2)
- added C11: 100nF, Capacitor_SMD:C_0402_1005Metric_Pad0.74x0.62mm_HandSolder, F.Cu at (181.3, 132.8)
- added C12: 100nF, Capacitor_SMD:C_0402_1005Metric_Pad0.74x0.62mm_HandSolder, F.Cu at (181.3, 131.8)
- added C13: 100nF, Capacitor_SMD:C_0402_1005Metric_Pad0.74x0.62mm_HandSolder, F.Cu at (190.2, 137.3)
- added C14: 100nF, Capacitor_SMD:C_0402_1005Metric_Pad0.74x0.62mm_HandSolder, F.Cu at (191.2, 136.2)
- added C16: 1uF, Capacitor_SMD:C_0402_1005Metric_Pad0.74x0.62mm_HandSolder, F.Cu at (213.7, 139.6)
- added C17: 100nF, Capacitor_SMD:C_0402_1005Metric_Pad0.74x0.62mm_HandSolder, F.Cu at (212.2, 139.6)
- added C19: 15pF, Capacitor_SMD:C_0402_1005Metric_Pad0.74x0.62mm_HandSolder, F.Cu at (223.9, 133.8)
- added C2: 15pF, Capacitor_SMD:C_0402_1005Metric_Pad0.74x0.62mm_HandSolder, F.Cu at (185.8, 145.6)
- added C20: 15pF, Capacitor_SMD:C_0402_1005Metric_Pad0.74x0.62mm_HandSolder, F.Cu at (224.5, 139.5)
- added C21: 1uF, Capacitor_SMD:C_0402_1005Metric_Pad0.74x0.62mm_HandSolder, F.Cu at (219.5, 140.2)
- added C22: 100nF, Capacitor_SMD:C_0402_1005Metric_Pad0.74x0.62mm_HandSolder, F.Cu at (220.5, 140.2)
- added C23: 1uF, Capacitor_SMD:C_0402_1005Metric_Pad0.74x0.62mm_HandSolder, F.Cu at (222.6, 140.2)
- added C24: 100nF, Capacitor_SMD:C_0402_1005Metric_Pad0.74x0.62mm_HandSolder, F.Cu at (221.6, 140.2)
- added C5: 100nF, Capacitor_SMD:C_0402_1005Metric_Pad0.74x0.62mm_HandSolder, F.Cu at (187.5, 145.8)
- added C6: 4.7uF, Capacitor_SMD:C_0402_1005Metric_Pad0.74x0.62mm_HandSolder, F.Cu at (188.5, 137.1)
- added C7: 10uF, Capacitor_SMD:C_0402_1005Metric_Pad0.74x0.62mm_HandSolder, F.Cu at (188.7, 133.5)
- added C8: 100nF, Capacitor_SMD:C_0402_1005Metric_Pad0.74x0.62mm_HandSolder, F.Cu at (177.1, 136.8)
- added C9: 100nF, Capacitor_SMD:C_0402_1005Metric_Pad0.74x0.62mm_HandSolder, F.Cu at (188.5, 142.2)
- added H1: MountingHole, MountingHole:MountingHole_3.2mm_M3, F.Cu at (64.8, 132.9)
- added H2: MountingHole, MountingHole:MountingHole_3.2mm_M3, F.Cu at (312.6, 139.0)
- added H3: MountingHole, MountingHole:MountingHole_3.2mm_M3, F.Cu at (235.3, 137.6)
- added J1: USB_C_Receptacle_USB2.0_14P, Connector_USB:USB_C_Receptacle_HRO_TYPE-C-31-M-12, F.Cu at (203.7, 130.1)
- added J2: Conn_01x05_Socket, imports:pogo 5pin 2.54, F.Cu at (73.7, 149.0)
- added J3: Conn_01x05_Socket, imports:pogo 5pin 2.54, F.Cu at (123.7, 149.0)
- added J4: Conn_01x05_Socket, imports:pogo 5pin 2.54, F.Cu at (173.7, 149.0)
- added J5: Conn_01x05_Socket, imports:pogo 5pin 2.54, F.Cu at (223.7, 149.0)
- added J6: Conn_01x05_Socket, imports:pogo 5pin 2.54, F.Cu at (273.6, 149.0)
- added J7: Conn_01x05_Socket, imports:pogo 5pin 2.54, F.Cu at (323.6, 149.0)
- added L1: 3.3uF, imports:INDC1608X95N, F.Cu at (188.9, 132.2)
- added R1: 1kR, Resistor_SMD:R_0402_1005Metric_Pad0.72x0.64mm_HandSolder, F.Cu at (184.2, 145.0)
- added R10: 5k1R, Resistor_SMD:R_0402_1005Metric_Pad0.72x0.64mm_HandSolder, F.Cu at (211.1, 130.6)
- added R2: 33R, Resistor_SMD:R_0402_1005Metric_Pad0.72x0.64mm_HandSolder, F.Cu at (188.7, 134.5)
- added R3: 27R, Resistor_SMD:R_0402_1005Metric_Pad0.72x0.64mm_HandSolder, F.Cu at (182.9, 129.5)
- added R4: 27R, Resistor_SMD:R_0402_1005Metric_Pad0.72x0.64mm_HandSolder, F.Cu at (184.0, 129.5)
- added R5: 10kR, Resistor_SMD:R_0402_1005Metric_Pad0.72x0.64mm_HandSolder, F.Cu at (177.8, 134.3)
- added R6: 1kR, Resistor_SMD:R_0402_1005Metric_Pad0.72x0.64mm_HandSolder, F.Cu at (169.2, 133.7)
- added R7: 10kR, Resistor_SMD:R_0402_1005Metric_Pad0.72x0.64mm_HandSolder, F.Cu at (193.6, 136.8)
- added R8: 1kR, Resistor_SMD:R_0402_1005Metric_Pad0.72x0.64mm_HandSolder, F.Cu at (192.8, 131.0)
- added R9: 5k1R, Resistor_SMD:R_0402_1005Metric_Pad0.72x0.64mm_HandSolder, F.Cu at (211.1, 129.6)
- added U3: SL2.1S, easyeda2kicad:SSOP-16_L4.6-W2.6-P0.53-LS4.0-BL, F.Cu at (217.7, 136.7)
- added USB1: TYPE-A-AF90, easyeda2kicad:USB-A-TH_U-A-24DD-Y-13, F.Cu at (323.8, 139.1)
- added USB2: TYPE-A-AF90, easyeda2kicad:USB-A-TH_U-A-24DD-Y-13, F.Cu at (343.5, 139.1)
- added USB3: TYPE-A-AF90, easyeda2kicad:USB-A-TH_U-A-24DD-Y-13, F.Cu at (333.6, 139.1)
- added Y1: ABM8-272-T3, Crystal:Crystal_SMD_Abracon_ABM8G-4Pin_3.2x2.5mm, F.Cu at (181.9, 144.5)
- added Y2: ABM8-272-T3, Crystal:Crystal_SMD_Abracon_ABM8G-4Pin_3.2x2.5mm, F.Cu at (224.2, 136.8)
- added boot: BOOTSEL, Button_Switch_SMD:SW_Push_SPST_NO_Alps_SKRK, F.Cu at (173.2, 133.7)
- added rst: RESET, Button_Switch_SMD:SW_Push_SPST_NO_Alps_SKRK, F.Cu at (195.5, 133.4)
- C3, C4: value 15pF -> 4.7uF
- D1: footprint Diode_SMD:D_0402_1005Metric_Pad0.77x0.64mm_HandSolder -> Diode_SMD:D_SOD-323
- D2, D3, D4: footprint Diode_SMD:D_0402_1005Metric_Pad0.77x0.64mm_HandSolder -> Diode_SMD:D_SOD-323; moved to B.Cu
- U5: renamed from U4; moved to B.Cu
- U6: renamed from U5; moved to B.Cu
- U7: renamed from U6; moved to B.Cu
- moved U6 368.2 mm to (343.4, 145.2), turned to 90 degrees
- moved D3 361.4 mm to (343.5, 132.3), turned to 90 degrees
- moved U7 357.8 mm to (333.5, 145.2), turned to 90 degrees
- moved U5 351.5 mm to (323.8, 145.2), turned to 90 degrees
- moved D4 351.5 mm to (333.6, 132.3), turned to 90 degrees
- moved D2 343.9 mm to (323.8, 132.3), turned to 90 degrees
- moved U4 246.1 mm to (207.1, 136.7)
- moved D1 239.3 mm to (201.3, 137.9), turned to 90 degrees
- moved C15 234.4 mm to (198.8, 137.5), turned to -90 degrees
- moved C18 233.2 mm to (197.8, 138.9), turned to -90 degrees
- moved U2 228.9 mm to (196.3, 136.9)
- moved C3 218.5 mm to (185.7, 132.4)
- moved C4 216.7 mm to (185.7, 131.4)
- moved U1 213.4 mm to (183.2, 137.9)
- renumbered C1 to C15, C2 to C18, U7 to U2, U3 to U4
Connections:
- C3 pad 1: GND -> +3V3
- C3 pad 2: /usb + power/USBHUB_XIN -> GND
- C4 pad 1: GND -> +1V1
- C4 pad 2: /usb + power/USBHUB_XOUT -> GND
- U1 pad 1: unconnected-(U1-IOVDD-Pad1) -> +3V3
- U1 pad 10: unconnected-(U1-GPIO7-Pad10) -> /i2c connections/BUS2_EN
- U1 pad 11: unconnected-(U1-IOVDD-Pad11) -> +3V3
- U1 pad 12: unconnected-(U1-GPIO8-Pad12) -> /i2c connections/BUS2_SDA
- U1 pad 13: unconnected-(U1-GPIO9-Pad13) -> /i2c connections/BUS2_SCL
- U1 pad 15: unconnected-(U1-GPIO11-Pad15) -> /i2c connections/BUS3_EN
- U1 pad 16: unconnected-(U1-GPIO12-Pad16) -> /i2c connections/BUS3_SDA
- U1 pad 17: unconnected-(U1-GPIO13-Pad17) -> /i2c connections/BUS3_SCL
- U1 pad 20: unconnected-(U1-IOVDD-Pad20) -> +3V3
- U1 pad 21: unconnected-(U1-XIN-Pad21) -> /RP_XIN
- U1 pad 22: unconnected-(U1-XOUT-Pad22) -> /RP_XOUT
- U1 pad 23: unconnected-(U1-DVDD-Pad23) -> +1V1
- U1 pad 26: unconnected-(U1-RUN-Pad26) -> /RESET
- U1 pad 27: unconnected-(U1-GPIO16-Pad27) -> /i2c connections/BUS4_EN
- U1 pad 28: unconnected-(U1-GPIO17-Pad28) -> /i2c connections/BUS4_SDA
- U1 pad 29: unconnected-(U1-GPIO18-Pad29) -> /i2c connections/BUS4_SCL
- U1 pad 30: unconnected-(U1-IOVDD-Pad30) -> +3V3
- U1 pad 31: unconnected-(U1-GPIO19-Pad31) -> /i2c connections/BUS5_EN
- U1 pad 32: unconnected-(U1-GPIO20-Pad32) -> /i2c connections/BUS5_SDA
- U1 pad 33: unconnected-(U1-GPIO21-Pad33) -> /i2c connections/BUS5_SCL
- U1 pad 34: unconnected-(U1-GPIO22-Pad34) -> /i2c connections/BUS6_EN
- U1 pad 35: unconnected-(U1-GPIO23-Pad35) -> /i2c connections/BUS6_SDA
- U1 pad 36: unconnected-(U1-GPIO24-Pad36) -> /i2c connections/BUS6_SCL
- U1 pad 38: unconnected-(U1-IOVDD-Pad38) -> +3V3
- U1 pad 39: unconnected-(U1-DVDD-Pad39) -> +1V1
- U1 pad 44: unconnected-(U1-ADC_AVDD-Pad44) -> +3V3
- U1 pad 45: unconnected-(U1-IOVDD-Pad45) -> +3V3
- U1 pad 46: unconnected-(U1-VREG_AVDD-Pad46) -> Net-(U1-VREG_AVDD)
- U1 pad 47: unconnected-(U1-VREG_PGND-Pad47) -> GND
- U1 pad 48: unconnected-(U1-VREG_LX-Pad48) -> /VREG_LX
- U1 pad 49: unconnected-(U1-VREG_VIN-Pad49) -> +3V3
- U1 pad 5: unconnected-(U1-GPIO3-Pad5) -> /i2c connections/BUS1_EN
- U1 pad 50: unconnected-(U1-VREG_FB-Pad50) -> +1V1
- U1 pad 51: unconnected-(U1-USB_DM-Pad51) -> Net-(U1-USB_DM)
- U1 pad 52: unconnected-(U1-USB_DP-Pad52) -> Net-(U1-USB_DP)
- U1 pad 53: unconnected-(U1-USB_OTP_VDD-Pad53) -> +3V3
- U1 pad 54: unconnected-(U1-QSPI_IOVDD-Pad54) -> +3V3
- U1 pad 6: unconnected-(U1-DVDD-Pad6) -> +1V1
- U1 pad 60: unconnected-(U1-QSPI_SS-Pad60) -> /BOOTSEL
- U1 pad 61: unconnected-(U1-GND-Pad61) -> GND
- U1 pad 7: unconnected-(U1-GPIO4-Pad7) -> /i2c connections/BUS1_SDA
- U1 pad 8: unconnected-(U1-GPIO5-Pad8) -> /i2c connections/BUS1_SCL
Routing:
- net +3V3: track 0.00 -> 352.7 mm, vias 0 -> 20
- net VSYS: track 0.00 -> 166.6 mm, vias 0 -> 9
- net /usb + power/PROT_USB2_D+: track 0.00 -> 153.7 mm, vias 0 -> 1
- net /usb + power/PROT_USB2_D-: track 0.00 -> 153.5 mm, vias 0 -> 1
- net /i2c connections/BUS6_SCL: track 0.00 -> 152.0 mm
- net /i2c connections/BUS6_SDA: track 0.00 -> 149.3 mm
- net /i2c connections/BUS6_EN: track 0.00 -> 146.7 mm
- net /usb + power/PROT_USB3_D-: track 0.00 -> 133.1 mm, vias 0 -> 1
- net /usb + power/PROT_USB3_D+: track 0.00 -> 131.8 mm, vias 0 -> 1
- net /usb + power/PROT_USB1_D-: track 0.00 -> 122.3 mm, vias 0 -> 1
- net /usb + power/PROT_USB1_D+: track 0.00 -> 121.1 mm, vias 0 -> 1
- net /i2c connections/BUS1_EN: track 0.00 -> 109.2 mm
- net /i2c connections/BUS1_SDA: track 0.00 -> 106.6 mm
- net /i2c connections/BUS1_SCL: track 0.00 -> 103.9 mm
- net /i2c connections/BUS5_SCL: track 0.00 -> 101.6 mm
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- added copper zone on B.Cu, net GND
- added copper zone on F.Cu, net GND
Other:
- board outline added: 290 x 24 mm

Commit message: finished all pcbs
Parts:
- added R11: 10kR, Resistor_SMD:R_0402_1005Metric_Pad0.72x0.64mm_HandSolder, F.Cu at (308.8, 141.5)
- added R12: 10kR, Resistor_SMD:R_0402_1005Metric_Pad0.72x0.64mm_HandSolder, F.Cu at (306.8, 141.5)
- added R13: 10kR, Resistor_SMD:R_0402_1005Metric_Pad0.72x0.64mm_HandSolder, F.Cu at (266.7, 145.8)
- added R14: 10kR, Resistor_SMD:R_0402_1005Metric_Pad0.72x0.64mm_HandSolder, F.Cu at (266.7, 143.8)
- added R15: 10kR, Resistor_SMD:R_0402_1005Metric_Pad0.72x0.64mm_HandSolder, F.Cu at (236.1, 145.4)
- added R16: 10kR, Resistor_SMD:R_0402_1005Metric_Pad0.72x0.64mm_HandSolder, F.Cu at (234.1, 145.4)
- added R17: 10kR, Resistor_SMD:R_0402_1005Metric_Pad0.72x0.64mm_HandSolder, F.Cu at (170.2, 144.4)
- added R18: 10kR, Resistor_SMD:R_0402_1005Metric_Pad0.72x0.64mm_HandSolder, F.Cu at (170.2, 142.4)
- added R19: 10kR, Resistor_SMD:R_0402_1005Metric_Pad0.72x0.64mm_HandSolder, F.Cu at (139.7, 145.6)
- added R20: 10kR, Resistor_SMD:R_0402_1005Metric_Pad0.72x0.64mm_HandSolder, F.Cu at (137.7, 145.6)
- added R21: 10kR, Resistor_SMD:R_0402_1005Metric_Pad0.72x0.64mm_HandSolder, F.Cu at (93.0, 145.0)
- added R22: 10kR, Resistor_SMD:R_0402_1005Metric_Pad0.72x0.64mm_HandSolder, F.Cu at (91.1, 145.0)
- renumbered boot to SW1, rst to SW2
Connections:
- C10 pad 2: GND -> unconnected-(C10-Pad2)
- C11 pad 2: GND -> unconnected-(C11-Pad2)
- C12 pad 2: GND -> unconnected-(C12-Pad2)
- C13 pad 2: GND -> unconnected-(C13-Pad2)
Routing:
- net +3V3: track 352.7 -> 391.3 mm, vias 20 -> 26
- net /i2c connections/BUS4_SCL: track 49.1 -> 62.7 mm
- net /i2c connections/BUS3_SCL: track 12.1 -> 21.3 mm, vias 0 -> 2
- net /i2c connections/BUS5_SCL: track 101.6 -> 110.7 mm, vias 0 -> 2
- net /i2c connections/BUS1_SCL: track 103.9 -> 112.8 mm
- net /i2c connections/BUS3_SDA: track 11.0 -> 19.2 mm, vias 0 -> 2
- net /i2c connections/BUS1_SDA: track 106.6 -> 114.3 mm, vias 0 -> 2
- net /i2c connections/BUS4_SDA: track 47.1 -> 54.3 mm
- net /i2c connections/BUS2_SDA: track 56.0 -> 61.5 mm, vias 0 -> 2
- net /i2c connections/BUS5_SDA: track 98.9 -> 104.3 mm, vias 0 -> 2
- net /i2c connections/BUS2_SCL: track 53.4 -> 58.3 mm
- net /i2c connections/BUS6_SDA: track 149.3 -> 153.2 mm, vias 0 -> 2
- net /i2c connections/BUS6_SCL: track 152.0 -> 154.7 mm
- net unconnected-(C10-Pad2): track 0.00 -> 1.69 mm, vias 0 -> 1
- net GND: track 15.5 -> 13.8 mm, vias 254 -> 250
