File: modules/controller_hub/pcb/i2c.kicad_sch (KiCad schematic)
At the start: 5 parts, among them J2 Conn_01x05_Socket, J3 Conn_01x05_Socket, J4 Conn_01x05_Socket, J5 Conn_01x05_Socket, J6 Conn_01x05_Socket

Commit message: add template for each module
Parts:
- added J7: Conn_01x05_Socket, symbol Connector:Conn_01x05_Socket
Connections:
- net +3V3: now also J7.1 (Pin_1)
- net BUS1_EN: now also J2.2 (Pin_2); no longer J2.3 (Pin_3)
- net BUS1_SDA: now also J2.3 (Pin_3); no longer J2.2 (Pin_2)
- net BUS2_EN: now also J4.2 (Pin_2); no longer J4.3 (Pin_3)
- net BUS2_SDA: now also J4.3 (Pin_3); no longer J4.2 (Pin_2)
- net BUS3_EN: now also J3.2 (Pin_2); no longer J3.3 (Pin_3)
- net BUS3_SDA: now also J3.3 (Pin_3); no longer J3.2 (Pin_2)
- net BUS4_EN: now also J5.2 (Pin_2); no longer J5.3 (Pin_3)
- net BUS4_SDA: now also J5.3 (Pin_3); no longer J5.2 (Pin_2)
- net BUS5_EN: now also J6.2 (Pin_2); no longer J6.3 (Pin_3)
- net BUS5_SDA: now also J6.3 (Pin_3); no longer J6.2 (Pin_2)
- net GND: now also J7.5 (Pin_5)
- new net BUS6_EN: J7.2 (Pin_2)
- new net BUS6_SCL: J7.4 (Pin_4)
- new net BUS6_SDA: J7.3 (Pin_3)

Commit message: hub done, started macropad
Parts:
- J2, J5, J6, J7: footprint (none) -> imports:pogo 5pin 2.54
- J3: renamed from J4; footprint (none) -> imports:pogo 5pin 2.54
- J4: renamed from J3; footprint (none) -> imports:pogo 5pin 2.54
Changed lines of the file:
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@@
 		(dnp no)
 		(fields_autoplaced yes)
-		(property "Reference" "#PWR041"
+		(property "Reference" "#PWR043"
 			(at 133.35 31.75 0)
 			(effects
@@
 			(project "CybdoKeebs_hub"
 				(path "/9919a4c0-a87a-4146-b547-4b221dff87d5/41905d77-ea62-40a6-b487-afb85a02e37c"
-					(reference "#PWR041")
+					(reference "#PWR043")
 					(unit 1)
 				)
@@
 			)
 		)
-		(property "Footprint" ""
+		(property "Footprint" "imports:pogo 5pin 2.54"
 			(at 140.97 35.56 0)
 			(effects
@@
 			)
 		)
-		(property "Footprint" ""
+		(property "Footprint" "imports:pogo 5pin 2.54"
 			(at 46.99 36.83 0)
 			(effects
@@
 		(dnp no)
 		(fields_autoplaced yes)
-		(property "Reference" "#PWR037"
+		(property "Reference" "#PWR039"
 			(at 86.36 33.02 0)
 			(effects
@@
 			(project "CybdoKeebs_hub"
 				(path "/9919a4c0-a87a-4146-b547-4b221dff87d5/41905d77-ea62-40a6-b487-afb85a02e37c"
-					(reference "#PWR037")
+					(reference "#PWR039")
 					(unit 1)
 				)
@@
 		(dnp no)
 		(fields_autoplaced yes)
-		(property "Reference" "#PWR040"
+		(property "Reference" "#PWR042"
 			(at 86.36 82.55 0)
 			(effects
@@
 			(project "CybdoKeebs_hub"
 				(path "/9919a4c0-a87a-4146-b547-4b221dff87d5/41905d77-ea62-40a6-b487-afb85a02e37c"
-					(reference "#PWR040")
+					(reference "#PWR042")
 					(unit 1)
 				)
@@
 		(dnp no)
 		(fields_autoplaced yes)
-		(property "Reference" "J3"
+		(property "Reference" "J4"
 			(at 95.25 35.5599 0)
 			(effects
@@
 			)
 		)
-		(property "Footprint" ""
+		(property "Footprint" "imports:pogo 5pin 2.54"
 			(at 93.98 36.83 0)
 			(effects
@@
 			(project "CybdoKeebs_hub"
 				(path "/9919a4c0-a87a-4146-b547-4b221dff87d5/41905d77-ea62-40a6-b487-afb85a02e37c"
-					(reference "J3")
+					(reference "J4")
 					(unit 1)
 				)
@@
 		(dnp no)
 		(fields_autoplaced yes)
-		(property "Reference" "J4"
+		(property "Reference" "J3"
 			(at 48.26 67.3099 0)
 			(effects
@@
 			)
 		)
-		(property "Footprint" ""
+		(property "Footprint" "imports:pogo 5pin 2.54"
 			(at 46.99 68.58 0)
 			(effects
@@
 			(project "CybdoKeebs_hub"
 				(path "/9919a4c0-a87a-4146-b547-4b221dff87d5/41905d77-ea62-40a6-b487-afb85a02e37c"
-					(reference "J4")
+					(reference "J3")
 					(unit 1)
 				)
@@
 		(dnp no)
 		(fields_autoplaced yes)
-		(property "Reference" "#PWR039"
+		(property "Reference" "#PWR041"
 			(at 86.36 64.77 0)
 			(effects
@@
 			(project "CybdoKeebs_hub"
 				(path "/9919a4c0-a87a-4146-b547-4b221dff87d5/41905d77-ea62-40a6-b487-afb85a02e37c"
-					(reference "#PWR039")
+					(reference "#PWR041")
 					(unit 1)
 				)
@@
 		(dnp no)
 		(fields_autoplaced yes)
-		(property "Reference" "#PWR034"
+		(property "Reference" "#PWR037"
 			(at 39.37 64.77 0)
 			(effects
@@
 			(project "CybdoKeebs_hub"
 				(path "/9919a4c0-a87a-4146-b547-4b221dff87d5/41905d77-ea62-40a6-b487-afb85a02e37c"
-					(reference "#PWR034")
+					(reference "#PWR037")
 					(unit 1)
 				)
@@
 		(dnp no)
 		(fields_autoplaced yes)
-		(property "Reference" "#PWR038"
+		(property "Reference" "#PWR040"
 			(at 86.36 50.8 0)
 			(effects
@@
 			(project "CybdoKeebs_hub"
 				(path "/9919a4c0-a87a-4146-b547-4b221dff87d5/41905d77-ea62-40a6-b487-afb85a02e37c"
-					(reference "#PWR038")
+					(reference "#PWR040")
 					(unit 1)
 				)
@@
 		(dnp no)
 		(fields_autoplaced yes)
-		(property "Reference" "#PWR033"
+		(property "Reference" "#PWR038"
 			(at 39.37 82.55 0)
 			(effects
@@
 			(project ""
 				(path "/9919a4c0-a87a-4146-b547-4b221dff87d5/41905d77-ea62-40a6-b487-afb85a02e37c"
-					(reference "#PWR033")
+					(reference "#PWR038")
 					(unit 1)
 				)
@@
 		(dnp no)
 		(fields_autoplaced yes)
-		(property "Reference" "#PWR042"
+		(property "Reference" "#PWR044"
 			(at 133.35 49.53 0)
 			(effects
@@
 			(project "CybdoKeebs_hub"
 				(path "/9919a4c0-a87a-4146-b547-4b221dff87d5/41905d77-ea62-40a6-b487-afb85a02e37c"
-					(reference "#PWR042")
+					(reference "#PWR044")
 					(unit 1)
 				)
@@
 			)
 		)
-		(property "Footprint" ""
+		(property "Footprint" "imports:pogo 5pin 2.54"
 			(at 140.97 68.58 0)
 			(effects
@@
 			)
 		)
-		(property "Footprint" ""
+		(property "Footprint" "imports:pogo 5pin 2.54"
 			(at 93.98 68.58 0)
 			(effects
