File: modules/controller_hub/pcb/usb_and_power.kicad_sch (KiCad schematic)
At the start: 27 parts, among them J1 USB_C_Receptacle_USB2.0_14P, U2 SL2.1S, U3 USBLC6-2P6, U4 USBLC6-2P6, U5 USBLC6-2P6, U6 USBLC6-2P6, U7 MCP1700x-300xxTT, Y1 ABM8-272-T3

Commit message: hub done, started macropad
Parts:
- removed C3, C4: 15pF, Capacitor_SMD:C_0402_1005Metric_Pad0.74x0.62mm_HandSolder, symbol Device:C
- removed Y1: ABM8-272-T3, symbol Device:Crystal_GND24
- added C19, C20: 15pF, Capacitor_SMD:C_0402_1005Metric_Pad0.74x0.62mm_HandSolder, symbol Device:C
- added Y2: ABM8-272-T3, Crystal:Crystal_SMD_Abracon_ABM8G-4Pin_3.2x2.5mm, symbol Device:Crystal_GND24
- J1: footprint (none) -> Connector_USB:USB_C_Receptacle_HRO_TYPE-C-31-M-12
- R10: renamed from R1; footprint (none) -> Resistor_SMD:R_0402_1005Metric_Pad0.72x0.64mm_HandSolder
- R9: renamed from R2; footprint (none) -> Resistor_SMD:R_0402_1005Metric_Pad0.72x0.64mm_HandSolder
- renumbered C1 to C15, C22 to C16, C23 to C17, C2 to C18, C26 to C21, C27 to C22, C24 to C23, C25 to C24, U7 to U2, U2 to U3, U3 to U4, U4 to U5, U5 to U6, U6 to U7, USB3 to USB1, USB1 to USB2, USB2 to USB3
Connections:
- net GND: now also C19.1, C20.1, Y2.2, Y2.4
- net PROT_USB1_D+: now also U3.14 (DP4); no longer U3.4 (DP1)
- net PROT_USB1_D-: now also U3.13 (DM4); no longer U3.3 (DM1)
- net USBHUB_XIN: now also C19.2, Y2.3
- net USBHUB_XOUT: now also C20.2, Y2.1
- net USB_RP_D+: now also U3.4 (DP1); no longer U3.14 (DP4)
- net USB_RP_D-: now also U3.3 (DM1); no longer U3.13 (DM4)
- net at J1.A5 (CC1): now also R10.1; no longer R9.1
- net at J1.B5 (CC2): now also R9.1; no longer R10.1
Other:
- moved on the sheet: R10, R9
