File: modules/template/PCB/cybdokeebs_template.kicad_pcb (KiCad board)
At the start: 2 copper layers, 1 part, among them U1 TCA4307DGKR

Commit message: ship ship ship!!!
Parts:
- added C1: 0.1uF, Capacitor_SMD:C_0402_1005Metric_Pad0.74x0.62mm_HandSolder, F.Cu at (33.9, 52.0)
- added C10: 100nF, Capacitor_SMD:C_0402_1005Metric_Pad0.74x0.62mm_HandSolder, F.Cu at (37.2, 57.9)
- added C11: 100nF, Capacitor_SMD:C_0402_1005Metric_Pad0.74x0.62mm_HandSolder, F.Cu at (37.2, 59.8)
- added C12: 100nF, Capacitor_SMD:C_0402_1005Metric_Pad0.74x0.62mm_HandSolder, F.Cu at (37.2, 61.8)
- added C13: 100nF, Capacitor_SMD:C_0402_1005Metric_Pad0.74x0.62mm_HandSolder, F.Cu at (40.4, 52.0)
- added C14: 100nF, Capacitor_SMD:C_0402_1005Metric_Pad0.74x0.62mm_HandSolder, F.Cu at (40.4, 53.9)
- added C15: 100nF, Capacitor_SMD:C_0402_1005Metric_Pad0.74x0.62mm_HandSolder, F.Cu at (40.4, 55.9)
- added C16: 100nF, Capacitor_SMD:C_0402_1005Metric_Pad0.74x0.62mm_HandSolder, F.Cu at (40.4, 57.9)
- added C17: 100nF, Capacitor_SMD:C_0402_1005Metric_Pad0.74x0.62mm_HandSolder, F.Cu at (40.4, 59.8)
- added C2: 0.1uF, Capacitor_SMD:C_0402_1005Metric_Pad0.74x0.62mm_HandSolder, F.Cu at (33.9, 53.9)
- added C3: 4.7uF, Capacitor_SMD:C_0402_1005Metric_Pad0.74x0.62mm_HandSolder, F.Cu at (33.9, 55.9)
- added C4: 4.7uF, Capacitor_SMD:C_0402_1005Metric_Pad0.74x0.62mm_HandSolder, F.Cu at (33.9, 57.9)
- added C5: 4.7uF, Capacitor_SMD:C_0402_1005Metric_Pad0.74x0.62mm_HandSolder, F.Cu at (33.9, 59.8)
- added C6: 4.7uF, Capacitor_SMD:C_0402_1005Metric_Pad0.74x0.62mm_HandSolder, F.Cu at (33.9, 61.8)
- added C7: 100nF, Capacitor_SMD:C_0402_1005Metric_Pad0.74x0.62mm_HandSolder, F.Cu at (37.2, 52.0)
- added C8: 100nF, Capacitor_SMD:C_0402_1005Metric_Pad0.74x0.62mm_HandSolder, F.Cu at (37.2, 53.9)
- added C9: 100nF, Capacitor_SMD:C_0402_1005Metric_Pad0.74x0.62mm_HandSolder, F.Cu at (37.2, 55.9)
- added J10: Conn_01x05_Pin, imports:pogo 5pin 2.54, F.Cu at (20.7, 43.5)
- added J11: Conn_01x05_Socket, imports:pogo 5pin 2.54, F.Cu at (20.7, 46.5)
- added J12: Conn_01x05_Socket, imports:pogo 5pin 2.54, F.Cu at (20.7, 49.5)
- added J13: Conn_01x05_Socket, imports:pogo 5pin 2.54, F.Cu at (20.7, 52.5)
- added J14: Conn_01x05_Socket, imports:pogo 5pin 2.54, F.Cu at (20.7, 55.5)
- added J15: Conn_01x05_Pin, imports:pogo 5pin 2.54, F.Cu at (20.7, 58.5)
- added J16: Conn_01x05_Pin, imports:pogo 5pin 2.54, F.Cu at (20.7, 61.5)
- added J9: Conn_01x05_Pin, imports:pogo 5pin 2.54, F.Cu at (20.7, 40.5)
- added L1: 3.3uF, imports:INDC1608X95N, F.Cu at (44.0, 59.1)
- added R1: 10kR, Resistor_SMD:R_0402_1005Metric_Pad0.72x0.64mm_HandSolder, F.Cu at (34.0, 40.0)
- added R10: 1kR, Resistor_SMD:R_0402_1005Metric_Pad0.72x0.64mm_HandSolder, F.Cu at (37.2, 46.0)
- added R2: 10kR, Resistor_SMD:R_0402_1005Metric_Pad0.72x0.64mm_HandSolder, F.Cu at (34.0, 42.0)
- added R3: 10kR, Resistor_SMD:R_0402_1005Metric_Pad0.72x0.64mm_HandSolder, F.Cu at (34.0, 44.0)
- added R4: 10kR, Resistor_SMD:R_0402_1005Metric_Pad0.72x0.64mm_HandSolder, F.Cu at (34.0, 46.0)
- added R5: 10kR, Resistor_SMD:R_0402_1005Metric_Pad0.72x0.64mm_HandSolder, F.Cu at (34.0, 48.0)
- added R6: 10kR, Resistor_SMD:R_0402_1005Metric_Pad0.72x0.64mm_HandSolder, F.Cu at (34.0, 50.0)
- added R7: 10kR, Resistor_SMD:R_0402_1005Metric_Pad0.72x0.64mm_HandSolder, F.Cu at (37.2, 40.0)
- added R8: 1kR, Resistor_SMD:R_0402_1005Metric_Pad0.72x0.64mm_HandSolder, F.Cu at (37.2, 42.0)
- added R9: 10kR, Resistor_SMD:R_0402_1005Metric_Pad0.72x0.64mm_HandSolder, F.Cu at (37.2, 44.0)
- added SW1: BOOTSEL, Button_Switch_SMD:SW_Push_SPST_NO_Alps_SKRK, F.Cu at (42.1, 41.3)
- added SW2: BOOTSEL, Button_Switch_SMD:SW_Push_SPST_NO_Alps_SKRK, F.Cu at (42.1, 45.7)
- added U2: RP2350_60QFN, RP2350_60QFN_minimal:RP2350-QFN-60-1EP_7x7_P0.4mm_EP3.4x3.4mm_ThermalVias, F.Cu at (23.1, 20.0)
- added U3: BM03B-SRSS-TB, easyeda2kicad:CONN-SMD-3P-P1.00_BM03B-SRSS-TB-LF-SN, F.Cu at (21.9, 27.7)
- U1: footprint easyeda:VSSOP-8_L3.0-W3.0-P0.65-LS4.9-BL -> easyeda2kicad:VSSOP-8_L3.0-W3.0-P0.65-LS4.9-BL
- moved U1 9.24 mm to (44.4, 54.4)
Connections:
- U1 pad 1: unconnected-(U1-EN-Pad1) -> Net-(U1-EN)
- U1 pad 2: unconnected-(U1-SCLOUT-Pad2) -> /minimum_system/SYS_SCL
- U1 pad 3: unconnected-(U1-SCLIN-Pad3) -> /minimum_system/0-0-SCL
- U1 pad 4: unconnected-(U1-GND-Pad4) -> GND
- U1 pad 5: unconnected-(U1-READY-Pad5) -> Net-(U1-READY)
- U1 pad 6: unconnected-(U1-SDAIN-Pad6) -> /minimum_system/0-0-SDA
- U1 pad 7: unconnected-(U1-SDAOUT-Pad7) -> /minimum_system/SYS_SDA
- U1 pad 8: unconnected-(U1-VCC-Pad8) -> +3V3
