File: modules/template/PCB/minimum_system.kicad_sch (KiCad schematic)
At the start: 41 parts, among them J10 Conn_01x05_Pin, J11 Conn_01x05_Socket, J12 Conn_01x05_Socket, J13 Conn_01x05_Socket, J14 Conn_01x05_Socket, J15 Conn_01x05_Pin, J16 Conn_01x05_Pin, J9 Conn_01x05_Pin, SW1 BOOTSEL, SW2 BOOTSEL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

Commit message: ship ship ship!!!
Parts:
- C1, C10, C11, C12, C13, C14, C15, C16, C17, C2, C3, C4, C5, C6, C7, C8, C9: footprint (none) -> Capacitor_SMD:C_0402_1005Metric_Pad0.74x0.62mm_HandSolder
- J10, J11, J12, J13, J14, J15, J16, J9: footprint (none) -> imports:pogo 5pin 2.54
- L1: footprint (none) -> imports:INDC1608X95N
- R1, R10, R2, R3, R4, R5, R6, R7, R8, R9: footprint (none) -> Resistor_SMD:R_0402_1005Metric_Pad0.72x0.64mm_HandSolder
- SW1, SW2: footprint (none) -> Button_Switch_SMD:SW_Push_SPST_NO_Alps_SKRK
- U1: footprint easyeda:VSSOP-8_L3.0-W3.0-P0.65-LS4.9-BL -> easyeda2kicad:VSSOP-8_L3.0-W3.0-P0.65-LS4.9-BL
